File: kb_pcb.kicad_sch (KiCad schematic)
At the start: 24 parts, among them SW1 SW_Push, U1 ATmega32U4-A, Y1 16MHz

Commit message: layout stuff
Parts:
- MX1, MX2, MX3, MX4: footprint MX_Alps_Hybrid:MX-10U-NoLED -> MX_Alps_Hybrid:MX-1U-NoLED
Changed lines of the file:
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@@
       (effects (font (size 0.508 0.508)))
     )
-    (property "Footprint" "MX_Alps_Hybrid:MX-10U-NoLED" (at 193.675 103.505 0)
+    (property "Footprint" "MX_Alps_Hybrid:MX-1U-NoLED" (at 193.675 103.505 0)
       (effects (font (size 1.524 1.524)) hide)
     )
@@
       (effects (font (size 0.508 0.508)))
     )
-    (property "Footprint" "MX_Alps_Hybrid:MX-10U-NoLED" (at 211.455 103.505 0)
+    (property "Footprint" "MX_Alps_Hybrid:MX-1U-NoLED" (at 211.455 103.505 0)
       (effects (font (size 1.524 1.524)) hide)
     )
@@
       (effects (font (size 0.508 0.508)))
     )
-    (property "Footprint" "MX_Alps_Hybrid:MX-10U-NoLED" (at 211.455 81.915 0)
+    (property "Footprint" "MX_Alps_Hybrid:MX-1U-NoLED" (at 211.455 81.915 0)
       (effects (font (size 1.524 1.524)) hide)
     )
@@
       (effects (font (size 0.508 0.508)))
     )
-    (property "Footprint" "MX_Alps_Hybrid:MX-10U-NoLED" (at 193.675 81.915 0)
-      (effects (font (size 1.524 1.524)) hide)
-    )
+    (property "Footprint" "MX_Alps_Hybrid:MX-1U-NoLED" (at 193.675 81.915 0)
+      (effects (font (size 1.524 1.524)) hide)
+    )

Commit message: schematic initial design
Parts:
- removed C3, C4: 0.1uF, Capacitor_SMD:C_0805_2012Metric, symbol Device:C_Small
- removed C5: 10uF, Capacitor_SMD:C_0805_2012Metric, symbol Device:C_Small
- removed C6, C7: 22pF, Capacitor_SMD:C_0805_2012Metric, symbol Device:C_Small
- removed F1: 500mA, Fuse:Fuse_1206_3216Metric, symbol Device:Polyfuse_Small
- removed R4: 10k, Resistor_SMD:R_0805_2012Metric, symbol Device:R_Small
- removed U1: ATmega32U4-A, Package_QFP:TQFP-44_10x10mm_P0.8mm, symbol MCU_Microchip_ATmega:ATmega32U4-A
- removed USB1: Molex-0548190589, random-keyboard-parts:Molex-0548190589, symbol random-keyboard-parts:Molex-0548190589
- added D10, D11, D12, D13, D14, D15, D16, D17, D18, D19, D20, D21, D22, D23, D24, D25, D26, D27, D28, D29, D30, D31, D32, D33, D34, D5, D6, D7, D8, D9: D_Small, symbol Device:D_Small
- added J1: USB_C_Receptacle, symbol Connector:USB_C_Receptacle
- added J3: AudioJack4, symbol Connector_Audio:AudioJack4
- added MX10, MX11, MX12, MX13, MX14, MX15, MX16, MX17, MX18, MX19, MX20, MX21, MX22, MX23, MX24, MX25, MX26, MX27, MX28, MX29, MX30, MX31, MX32, MX33, MX34, MX5, MX6, MX7, MX8, MX9: MX-NoLED, symbol MX_Alps_Hybrid:MX-NoLED
- added U1: RP2040, Package_DFN_QFN:QFN-56-1EP_7x7mm_P0.4mm_EP3.2x3.2mm, symbol MCU_RaspberryPi:RP2040
- C1: value 1uF -> 22pF; footprint Capacitor_SMD:C_0805_2012Metric -> (none)
- C2: value 0.1uF -> 22pF; footprint Capacitor_SMD:C_0805_2012Metric -> (none)
- D1, D2, D3, D4: value SOD-123 -> D_Small; footprint Diode_SMD:D_SOD-123 -> (none)
- MX1, MX2, MX3, MX4: footprint MX_Alps_Hybrid:MX-1U-NoLED -> (none)
- R1: value 10k -> 56k; footprint Resistor_SMD:R_0805_2012Metric -> (none)
- R2, R3: value 22 -> 56k; footprint Resistor_SMD:R_0805_2012Metric -> (none)
- SW1: footprint random-keyboard-parts:Reset_Pretty -> (none)
- Y1: footprint Crystal:Crystal_SMD_3225-4Pin_3.2x2.5mm -> (none)
Connections:
- net D+ is gone; now on net +5V: R2.1
- net D- is gone; now on net +5V: R3.1
- net ROW0 is gone; now on net ROW1: D1.1 (K), D2.1 (K)
- net +5V: now also R1.1, J3.T; no longer C2.1
- net COL1: now also MX1.1 (COL), MX13.1 (COL), MX19.1 (COL), MX27.1 (COL), MX7.1 (COL), U1.7 (GPIO5); no longer MX2.1 (COL), MX4.1 (COL)
- net GND: now also C1.1, C2.1, J1.A1 (GND), J1.A12 (GND), J1.B1 (GND), J1.B12 (GND), J1.S1 (SHIELD), J3.S, U1.19 (TESTEN), U1.57 (GND); no longer C2.2, R1.2
- net ROW1: now also D5.1 (K), D6.1 (K), U1.2 (GPIO0)
- net at SW1.2: now also R3.2, U1.26 (RUN)
- net at Y1.3: now also C2.2, U1.21 (XOUT)
- net at R2.2: now also J1.B5 (CC2), U1.39 (GPIO27_ADC1)
- net at Y1.1: now also C1.2, U1.20 (XIN)
- net COL0 renamed COL3
- net COL3: now also MX15.1 (COL), MX21.1 (COL), MX29.1 (COL), MX9.1 (COL), U1.9 (GPIO7); no longer MX1.1 (COL)
- new net: D9.2 (A), MX9.2 (ROW)
- new net: D21.2 (A), MX21.2 (ROW)
- new net: D16.2 (A), MX16.2 (ROW)
- new net: D15.2 (A), MX15.2 (ROW)
- new net: D14.2 (A), MX14.2 (ROW)
- new net: D30.2 (A), MX30.2 (ROW)
- new net: J3.R1, U1.36 (GPIO24)
- new net: J3.R2, U1.37 (GPIO25)
- new net: J1.A4 (VBUS), J1.A9 (VBUS), J1.B4 (VBUS), J1.B9 (VBUS), U1.48 (USB_VDD)
- new net: J1.A5 (CC1), R1.2, U1.38 (GPIO26_ADC0)
- new net: J1.A6 (D+), J1.B6 (D+), U1.47 (USB_DP)
- new net: J1.A7 (D-), J1.B7 (D-), U1.46 (USB_DM)
- new net: D27.2 (A), MX27.2 (ROW)
- new net: D18.2 (A), MX18.2 (ROW)
- new net: D28.2 (A), MX28.2 (ROW)
- new net: D22.2 (A), MX22.2 (ROW)
- new net: D17.2 (A), MX17.2 (ROW)
- new net: D34.2 (A), MX34.2 (ROW)
- new net: D24.2 (A), MX24.2 (ROW)
- new net: D19.2 (A), MX19.2 (ROW)
- new net: D12.2 (A), MX12.2 (ROW)
- new net: D31.2 (A), MX31.2 (ROW)
- new net: D13.2 (A), MX13.2 (ROW)
- new net: D33.2 (A), MX33.2 (ROW)
- new net: D8.2 (A), MX8.2 (ROW)
- new net: D5.2 (A), MX5.2 (ROW)
- new net: D7.2 (A), MX7.2 (ROW)
- new net: D20.2 (A), MX20.2 (ROW)
- new net: D6.2 (A), MX6.2 (ROW)
- new net: D10.2 (A), MX10.2 (ROW)
- new net: D25.2 (A), MX25.2 (ROW)
- new net: D26.2 (A), MX26.2 (ROW)
- new net: D32.2 (A), MX32.2 (ROW)
- new net: U1.1 (IOVDD), U1.10 (IOVDD), U1.22 (IOVDD), U1.33 (IOVDD), U1.42 (IOVDD), U1.49 (IOVDD)
- new net: U1.23 (DVDD), U1.50 (DVDD)
- new net: D29.2 (A), MX29.2 (ROW)
- new net: D23.2 (A), MX23.2 (ROW)
- new net: D11.2 (A), MX11.2 (ROW)
- new net COL2: MX14.1 (COL), MX2.1 (COL), MX20.1 (COL), MX28.1 (COL), MX8.1 (COL), U1.8 (GPIO6)
- new net COL4: MX10.1 (COL), MX16.1 (COL), MX22.1 (COL), MX30.1 (COL), MX4.1 (COL), U1.11 (GPIO8)
- new net COL5: MX11.1 (COL), MX17.1 (COL), MX23.1 (COL), MX31.1 (COL), MX5.1 (COL), U1.12 (GPIO9)
- new net COL6: MX12.1 (COL), MX18.1 (COL), MX24.1 (COL), MX32.1 (COL), MX6.1 (COL), U1.13 (GPIO10)
- new net COL7: MX25.1 (COL), MX26.1 (COL), MX33.1 (COL), MX34.1 (COL), U1.14 (GPIO11)
- new net ROW2: D10.1 (K), D11.1 (K), D12.1 (K), D34.1 (K), D7.1 (K), D8.1 (K), D9.1 (K), U1.3 (GPIO1)
- new net ROW3: D13.1 (K), D14.1 (K), D15.1 (K), D16.1 (K), D17.1 (K), D18.1 (K), D25.1 (K), U1.4 (GPIO2)
- new net ROW4: D19.1 (K), D20.1 (K), D21.1 (K), D22.1 (K), D23.1 (K), D24.1 (K), D26.1 (K), U1.5 (GPIO3)
- new net ROW5: D27.1 (K), D28.1 (K), D29.1 (K), D30.1 (K), D31.1 (K), D32.1 (K), D33.1 (K), U1.6 (GPIO4)
Other:
- company: (none) -> Matrix Studios
- title: (none) -> RV204034
